File: analog-noise-fob-sp23.brd (EAGLE design)
At the start: 110.6 x 77 mm, 10 parts

Commit message: autosaves
Parts:
- moved U$10 150.3 mm to (46.7, 91.9), turned to 270 degrees
- moved U$4 144.0 mm to (58.1, 78.7), turned to 90 degrees
- moved U$8 130.5 mm to (79.7, 77.4), turned to 180 degrees
- moved PH1 123.4 mm to (27.4, 85.7), turned to 270 degrees
- moved U$1 123.2 mm to (17.4, 69.3), turned to 270 degrees
- moved U$3 119.2 mm to (58.8, 50.0), turned to 0 degrees
- moved U$5 116.1 mm to (72.4, 35.3)
- moved U$2 96.2 mm to (52.5, 43.8), turned to 270 degrees
- moved U$6 57.8 mm to (52.2, 18.6), turned to 90 degrees
- moved U$7 40.7 mm to (52.0, 8.35), turned to 270 degrees
Routing:
- net N$2: track 78.3 -> 0.00 mm
- net N$6: track 52.7 -> 0.00 mm
- net N$5: track 48.7 -> 0.00 mm
- net N$3: track 31.7 -> 0.00 mm
- net N$1: track 26.1 -> 0.00 mm
- net N$4: track 8.05 -> 0.00 mm
Other:
- board size 110.6 x 77 mm -> 337.5 x 132.6 mm
